File: Gloves PCB.brd (EAGLE design)
At the start: 50.8 x 82.9 mm, 37 parts, among them U1 LM3914

Commit message: v1.1 commit
Parts:
- removed INPUTS: (no value), con-lsta:FE08-2W
- removed LED11, LED12: LP2C63-ST-RGB-SR0, led:LP2C63-ST-RGB-SR0
- removed OUTPUTS: (no value), con-lsta:FE05-2W
- removed R17, R18: 10R, rcl:R0402
- removed R19: 68R, rcl:R0402
- added J1, J2: MOLEX-53048-0810, x-io:MOLEX-53048-0810
- added J3: MOLEX-53048-0310, x-io:MOLEX-53048-0310
- added J4, J5, J6: MOLEX-53048-0210, x-io:MOLEX-53048-0210
- added JP1: M02-JST-2-PTH-NO_SILK, SparkFun-Connectors:JST-2-PTH-NS
- added S1: (no value), x-io:WURTH-ELEKTRONIK-450301014042
- R1, R10, R11, R12, R13, R14, R15, R16, R2, R3, R4, R5, R6, R7, R8, R9: device rcl:R0402 -> SparkFun-Passives:0805
- U1: value LM3914 -> LM3914V/NOPB; device x-io:DIL18 -> x-io:PLCC-20
- moved U$1 80.5 mm to (31.9, 3.02)
- moved R6 72.2 mm to (17.8, 79.4), flipped to the top, turned to 270 degrees
- moved R9 53.9 mm to (8.89, 15.9), flipped to the top
- moved R7 14.0 mm to (20.3, 79.4), flipped to the top, turned to 90 degrees
- moved R10 8.35 mm to (11.4, 15.9), flipped to the top, turned to 270 degrees
- moved R11 8.35 mm to (14.0, 15.9), flipped to the top, turned to 270 degrees
- moved R12 8.35 mm to (16.5, 15.9), flipped to the top, turned to 270 degrees
- moved R13 8.35 mm to (19.1, 15.9), flipped to the top, turned to 270 degrees
- moved R14 8.35 mm to (21.6, 15.9), flipped to the top, turned to 270 degrees
- moved R15 8.35 mm to (24.1, 15.9), flipped to the top, turned to 270 degrees
- moved R16 8.35 mm to (26.7, 15.9), flipped to the top, turned to 270 degrees
- moved R8 8.03 mm to (22.9, 79.4), flipped to the top
- moved U$2 5.08 mm to (17.8, 29.2)
- moved U$3 5.08 mm to (20.3, 69.8)
- moved R2 3.86 mm to (25.4, 77.5), flipped to the top
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Connections:
- removed net L_LED_B: LED11.3
- removed net L_LED_G: LED11.1
- removed net L_LED_GND: LED11.4, LED11.5, LED11.6
- removed net L_LED_R: LED11.2
- removed net N$17: OUTPUTS.4, R18.2
- removed net N$18: OUTPUTS.6, R17.2
- removed net OUT6: R18.1, U$2.31
- removed net OUT7: R17.1, U$2.30
- removed net R_LED_B: LED12.3
- removed net R_LED_G: LED12.1
- removed net R_LED_GND: LED12.4, LED12.5, LED12.6
- removed net R_LED_R: LED12.2
- removed net VBATT: LED1.A, LED10.A, LED2.A, LED3.A, LED4.A, LED5.A, LED6.A, LED7.A, LED8.A, LED9.A, R7.2, U$2.20, U1.3, U1.9
- removed net VDD: R10.1, R11.1, R12.1, R13.1, R14.1, R15.1, R16.1, R6.1, U$2.17, U$3.1
- new net 3V3: J3.2, R10.2, R11.2, R12.2, R13.2, R14.2, R15.2, R16.2, R9.2, U$2.17, U$3.1
- new net IN13: J6.1, U$2.13
- new net N$21: U$2.36, U$3.2
- new net VSUPPLY: LED1.A, LED10.A, LED2.A, LED3.A, LED4.A, LED5.A, LED6.A, LED7.A, LED8.A, LED9.A, R6.2, S1.2, U$2.20, U1.11, U1.3
- net GND: now also J2.1, J2.2, J2.3, J2.4, J2.5, J2.6, J2.7, J2.8, J3.3, J4.2, J5.2, J6.2, JP1.1; no longer INPUTS.1, INPUTS.11, INPUTS.13, INPUTS.15, INPUTS.3, INPUTS.5, INPUTS.7, INPUTS.9, OUTPUTS.1, OUTPUTS.3, OUTPUTS.5, OUTPUTS.7, OUTPUTS.9
- net IN10: now also J1.6, R14.1; no longer INPUTS.6, R14.2
- net IN11: now also J1.7, R15.1; no longer INPUTS.4, R15.2
- net IN12: now also J1.8, R16.1; no longer INPUTS.2, R16.2
- net IN5: now also J1.1, R9.1; no longer INPUTS.16, R6.2
- net IN6: now also J1.2, R10.1; no longer INPUTS.14, R10.2
- net IN7: now also J1.3, R11.1; no longer INPUTS.12, R11.2
- net IN8: now also J1.4, R12.1; no longer INPUTS.10, R12.2
- net IN9: now also J1.5, R13.1; no longer INPUTS.8, R13.2
- net N$10: now also U1.15; no longer U1.13
- net N$11: now also U1.16; no longer U1.14
- net N$12: now also U1.17; no longer U1.15
- net N$13: now also U1.18; no longer U1.16
- net N$14: now also U1.19; no longer U1.17
- net N$15: now also U1.20; no longer U1.18
- net N$3: now also JP1.2, S1.3; no longer OUTPUTS.2, R19.2
- net N$4: now also R7.1; no longer R9.1
- net N$5: now also R6.1, R7.2; no longer R7.1, R9.2
- net N$6: now also U1.10; no longer U1.8
- net N$7: now also U1.12; no longer U1.10
- net N$8: now also U1.13; no longer U1.11
- net N$9: now also U1.14; no longer U1.12
- net OUT5: now also J3.1; no longer R19.1
- net OUT8: now also J4.1; no longer OUTPUTS.8
- net OUT9: now also J5.1; no longer OUTPUTS.10
- net REF_OUT: now also U1.8; no longer U1.7
Routing:
- net VBATT: track 121.3 -> 0.00 mm
- net VSUPPLY: track 0.00 -> 114.8 mm
- net IN13: track 0.00 -> 41.1 mm
- net GND: track 0.00 -> 34.4 mm
- net N$13: track 40.4 -> 16.2 mm
- net VDD: track 22.4 -> 0.00 mm
- net OUT7: track 19.0 -> 0.00 mm
- net N$21: track 0.00 -> 17.4 mm
- net N$4: track 5.95 -> 22.7 mm
- net N$12: track 36.1 -> 20.6 mm
- net OUT6: track 14.9 -> 0.00 mm
- net N$3: track 1.89 -> 13.6 mm
- net R_LED_GND: track 9.91 -> 0.00 mm
- net L_LED_GND: track 9.91 -> 0.00 mm
- net L_LED_B: track 9.15 -> 0.00 mm
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- added copper zone on layer 1, net 3V3
- removed copper zone on layer 1, net L_LED_B
- removed copper zone on layer 1, net L_LED_G
- removed copper zone on layer 1, net L_LED_GND
- removed copper zone on layer 1, net L_LED_R
- removed copper zone on layer 16, net N$19
- removed copper zone on layer 16, net N$20
- removed copper zone on layer 1, net R_LED_B
- removed copper zone on layer 1, net R_LED_G
- removed copper zone on layer 1, net R_LED_GND
- removed copper zone on layer 1, net R_LED_R
- removed copper zone on layer 1, net VDD
Other:
- outline, holes or cut-outs redrawn
- board text added: "3V3"
- board text added: "BATTERY"
- board text added: "BUTTON"
- board text added: "Flex (Ground)"
- board text added: "Flex (Signal)"
- board text added: "Gloves PCB v1.1"
- board text added: "INPUTS"
- board text added: "MOT (L)"
- board text added: "MOT (R)"
- board text added: "OUTPUTS"
- board text added: "RGB"
- board text removed: "3V3 OUT"
- board text removed: "B"
- board text removed: "BATT"
- board text removed: "G"
- board text removed: "Gloves PCB v1.0"
- board text removed: "IN10"
- board text removed: "IN11"
- board text removed: "IN12"
- board text removed: "IN5"
- board text removed: "IN6"
- board text removed: "IN7"
- board text removed: "IN8"
- board text removed: "IN9"
- board text removed: "OUT5"
- board text removed: "OUT6"
- board text removed: "OUT7"
- board text removed: "OUT8"
- board text removed: "OUT9"
- board text removed: "R"
