File: Gloves PCB.sch (EAGLE design)
At the start: 37 parts, among them U1 LM3914

Commit message: v1.1 commit
Parts:
- removed INPUTS: (no value), con-lsta:FE08-2W
- removed LED11, LED12: LP2C63-ST-RGB-SR0, led:LP2C63-ST-RGB-SR0
- removed OUTPUTS: (no value), con-lsta:FE05-2W
- removed R17, R18: 10R, rcl:R-EU_R0402
- removed R19: 68R, rcl:R-EU_R0402
- added J1, J2: MOLEX-53048-0810, x-io:MOLEX-53048-0810
- added J3: MOLEX-53048-0310, x-io:MOLEX-53048-0310
- added J4, J5, J6: MOLEX-53048-0210, x-io:MOLEX-53048-0210
- added JP1: M02-JST-2-PTH-NO_SILK, SparkFun-Connectors:M02-JST-2-PTH-NO_SILK
- added S1: (no value), x-io:SWITCH-DPST
- R1, R10, R11, R12, R13, R14, R15, R16, R2, R3, R4, R5, R6, R7, R8, R9: device rcl:R-EU_R0402 -> SparkFun-Passives:RESISTOR0805-RES
- U1: value LM3914 -> LM3914V/NOPB; device x-io:LM3914 -> x-io:LM3914PLCC
Connections:
- removed net L_LED_B: LED11B.A
- removed net L_LED_G: LED11G.A
- removed net L_LED_GND: LED11B.C, LED11G.C, LED11R.C
- removed net L_LED_R: LED11R.A
- removed net N$17: OUTPUTS.4, R18.2
- removed net N$18: OUTPUTS.6, R17.2
- removed net OUT6: R18.1, U$2.OUT6
- removed net OUT7: R17.1, U$2.OUT7
- removed net R_LED_B: LED12B.A
- removed net R_LED_G: LED12G.A
- removed net R_LED_GND: LED12B.C, LED12G.C, LED12R.C
- removed net R_LED_R: LED12R.A
- removed net VBATT: LED1.A, LED10.A, LED2.A, LED3.A, LED4.A, LED5.A, LED6.A, LED7.A, LED8.A, LED9.A, R7.2, U$2.BATTERY, U1.MODE, U1.V+
- removed net VDD: R10.1, R11.1, R12.1, R13.1, R14.1, R15.1, R16.1, R6.1, U$2.3.3V-OUT, U$3.VDD
- new net 3V3: J3.2, R10.2, R11.2, R12.2, R13.2, R14.2, R15.2, R16.2, R9.2, U$2.3.3V-OUT, U$3.VDD
- new net IN13: J6.1, U$2.IN13
- new net N$21: U$2.OUT1, U$3.RX-INPUT
- new net VSUPPLY: LED1.A, LED10.A, LED2.A, LED3.A, LED4.A, LED5.A, LED6.A, LED7.A, LED8.A, LED9.A, R6.2, S1.2, U$2.BATTERY, U1.MODE, U1.V+
- net GND: now also J2.1, J2.2, J2.3, J2.4, J2.5, J2.6, J2.7, J2.8, J3.3, J4.2, J5.2, J6.2, JP1.1; no longer INPUTS.1, INPUTS.11, INPUTS.13, INPUTS.15, INPUTS.3, INPUTS.5, INPUTS.7, INPUTS.9, OUTPUTS.1, OUTPUTS.3, OUTPUTS.5, OUTPUTS.7, OUTPUTS.9
- net IN10: now also J1.6, R14.1; no longer INPUTS.6, R14.2
- net IN11: now also J1.7, R15.1; no longer INPUTS.4, R15.2
- net IN12: now also J1.8, R16.1; no longer INPUTS.2, R16.2
- net IN5: now also J1.1, R9.1; no longer INPUTS.16, R6.2
- net IN6: now also J1.2, R10.1; no longer INPUTS.14, R10.2
- net IN7: now also J1.3, R11.1; no longer INPUTS.12, R11.2
- net IN8: now also J1.4, R12.1; no longer INPUTS.10, R12.2
- net IN9: now also J1.5, R13.1; no longer INPUTS.8, R13.2
- net N$3: now also JP1.2, S1.3; no longer OUTPUTS.2, R19.2
- net N$4: now also R7.1; no longer R9.1
- net N$5: now also R6.1, R7.2; no longer R7.1, R9.2
- net OUT5: now also J3.1; no longer R19.1
- net OUT8: now also J4.1; no longer OUTPUTS.8
- net OUT9: now also J5.1; no longer OUTPUTS.10
Other:
- note removed: "LED R/G/B = OUT 5/6/7"
